File: castellated_breakout.kicad_sch (KiCad schematic)
At the start: 4 parts, among them J1 Conn_01x14_Female, J2 Conn_01x14_Female, J3 Conn_01x06_Female, U1 STM32_7x4_Castellated

Commit message: updates
Parts:
- J3: footprint Connector:Tag-Connect_TC2030-IDC-NL_2x03_P1.27mm_Vertical -> Connector:Tag-Connect_TC2030-IDC-FP_2x03_P1.27mm_Vertical
Changed lines of the file:
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@@
       (effects (font (size 1.27 1.27)) (justify left))
     )
-    (property "Footprint" "Connector:Tag-Connect_TC2030-IDC-NL_2x03_P1.27mm_Vertical" (id 2) (at 157.48 53.34 0)
+    (property "Footprint" "Connector:Tag-Connect_TC2030-IDC-FP_2x03_P1.27mm_Vertical" (id 2) (at 157.48 53.34 0)
       (effects (font (size 1.27 1.27)) hide)
     )
@@
     )
     (path "/00000000-0000-0000-0000-0000613cfd7b"
-      (reference "J3") (unit 1) (value "Conn_01x06_Female") (footprint "Connector:Tag-Connect_TC2030-IDC-NL_2x03_P1.27mm_Vertical")
+      (reference "J3") (unit 1) (value "Conn_01x06_Female") (footprint "Connector:Tag-Connect_TC2030-IDC-FP_2x03_P1.27mm_Vertical")
     )
     (path "/00000000-0000-0000-0000-000061003436"
